Commit message: Final: camera added, LiDAR fixed, clean SLAM map, office world

File: urdf/Office_delivery_bot2.urdf (robot description, URDF)
Before this commit: robot Office_delivery_bot2, 6 links, 5 joints
Links:
- added link camera_link, mass 0.05; collision box size=0.03 0.08 0.03; visual box size=0.03 0.08 0.03
Joints:
- added joint camera_joint: type fixed, parent base_link, child camera_link, origin xyz=0 -0.26 0.578 rpy=0 0 -1.5708
- joint Lidar_Joint: origin xyz=0 0.01 0.8 rpy=0 0 0 -> xyz=0 0.01 0.81 rpy=0 0 0
